File: GCU-ADU.kicad_pcb (KiCad board)
At the start: 2 copper layers, 48.6 x 32.4 mm, 5 parts, among them X1 SW_Push, Y1 SW_Push

Commit message: Update
- Update with proper switches
Parts:
- A1, B1, X1, Y1: footprint Button_Switch_SMD:SW_Push_1P1T_NO_6x6mm_H9.5mm -> ADU:EVQ-Q2F02W
Routing:
- net X1: track 90.4 -> 104.2 mm, vias 1 -> 2
- net X4: track 47.2 -> 49.2 mm
- net X5: track 19.6 -> 19.0 mm
Other:
- outline, holes or cut-outs redrawn
