File: GCU-ADU.kicad_sch (KiCad schematic)
At the start: 5 parts, among them X1 SW_Push, Y1 SW_Push

Commit message: Update
- Update with proper switches
Parts:
- A1, B1, X1, Y1: footprint Button_Switch_SMD:SW_Push_1P1T_NO_6x6mm_H9.5mm -> ADU:EVQ-Q2F02W; LCSC (none) -> C388887; MPN (none) -> EVQ-Q2F02W
Changed lines of the file:
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@@
 			)
 		)
-		(property "Footprint" "Button_Switch_SMD:SW_Push_1P1T_NO_6x6mm_H9.5mm"
+		(property "Footprint" "ADU:EVQ-Q2F02W"
 			(at 128.27 62.23 0)
 			(effects
@@
 			)
 		)
-		(property "Datasheet" "~"
+		(property "Datasheet" "https://www3.panasonic.biz/ac/cdn/e/control/switch/light-touch/catalog/sw_lt_eng_6s_th.pdf"
 			(at 128.27 62.23 0)
 			(effects
@@
 			)
 		)
-		(property "Description" "Push button switch, generic, two pins"
+		(property "Description" "1 million press, 2.5mm height tactile button"
+			(at 128.27 67.31 0)
+			(effects
+				(font
+					(size 1.27 1.27)
+				)
+				(hide yes)
+			)
+		)
+		(property "LCSC" "C388887"
+			(at 128.27 67.31 0)
+			(effects
+				(font
+					(size 1.27 1.27)
+				)
+				(hide yes)
+			)
+		)
+		(property "MPN" "EVQ-Q2F02W"
 			(at 128.27 67.31 0)
 			(effects
@@
 			)
 		)
+		(property "LCSC" ""
+			(at 85.09 46.99 0)
+			(effects
+				(font
+					(size 1.27 1.27)
+				)
+				(hide yes)
+			)
+		)
 		(pin "1"
 		)
@@
 			)
 		)
-		(property "Footprint" "Button_Switch_SMD:SW_Push_1P1T_NO_6x6mm_H9.5mm"
+		(property "Footprint" "ADU:EVQ-Q2F02W"
 			(at 128.27 52.07 0)
 			(effects
@@
 			)
 		)
-		(property "Datasheet" "~"
+		(property "Datasheet" "https://www3.panasonic.biz/ac/cdn/e/control/switch/light-touch/catalog/sw_lt_eng_6s_th.pdf"
 			(at 128.27 52.07 0)
 			(effects
@@
 			)
 		)
-		(property "Description" "Push button switch, generic, two pins"
+		(property "Description" "1 million press, 2.5mm height tactile button"
+			(at 128.27 57.15 0)
+			(effects
+				(font
+					(size 1.27 1.27)
+				)
+				(hide yes)
+			)
+		)
+		(property "LCSC" "C388887"
+			(at 128.27 57.15 0)
+			(effects
+				(font
+					(size 1.27 1.27)
+				)
+				(hide yes)
+			)
+		)
+		(property "MPN" "EVQ-Q2F02W"
 			(at 128.27 57.15 0)
 			(effects
@@
 			)
 		)
-		(property "Footprint" "Button_Switch_SMD:SW_Push_1P1T_NO_6x6mm_H9.5mm"
+		(property "Footprint" "ADU:EVQ-Q2F02W"
 			(at 128.27 41.91 0)
 			(effects
@@
 			)
 		)
-		(property "Datasheet" "~"
+		(property "Datasheet" "https://www3.panasonic.biz/ac/cdn/e/control/switch/light-touch/catalog/sw_lt_eng_6s_th.pdf"
 			(at 128.27 41.91 0)
 			(effects
@@
 			)
 		)
-		(property "Description" "Push button switch, generic, two pins"
+		(property "Description" "1 million press, 2.5mm height tactile button"
+			(at 128.27 46.99 0)
+			(effects
+				(font
+					(size 1.27 1.27)
+				)
+				(hide yes)
+			)
+		)
+		(property "LCSC" "C388887"
+			(at 128.27 46.99 0)
+			(effects
+				(font
+					(size 1.27 1.27)
+				)
+				(hide yes)
+			)
+		)
+		(property "MPN" "EVQ-Q2F02W"
 			(at 128.27 46.99 0)
 			(effects
@@
 			)
 		)
-		(property "Footprint" "Button_Switch_SMD:SW_Push_1P1T_NO_6x6mm_H9.5mm"
+		(property "Footprint" "ADU:EVQ-Q2F02W"
 			(at 128.27 72.39 0)
 			(effects
@@
 			)
 		)
-		(property "Datasheet" "~"
+		(property "Datasheet" "https://www3.panasonic.biz/ac/cdn/e/control/switch/light-touch/catalog/sw_lt_eng_6s_th.pdf"
 			(at 128.27 72.39 0)
 			(effects
@@
 			)
 		)
-		(property "Description" "Push button switch, generic, two pins"
+		(property "Description" "1 million press, 2.5mm height tactile button"
 			(at 128.27 77.47 0)
 			(effects
+				(font
+					(size 1.27 1.27)
+				)
+				(hide yes)
+			)
+		)
+		(property "LCSC" "C388887"
+			(at 128.27 77.47 0)
+			(effects
+				(font
+					(size 1.27 1.27)
+				)
+				(hide yes)
+			)
+		)
+		(property "MPN" "EVQ-Q2F02W"
+			(at 128.27 77.47 0)
+			(effects
